Commit message: guardian_terabot_description: Setting the correct position of the arm

File: guardian_terabot_description/robots/guardian_terabot.urdf.xacro (robot description, xacro)
@@ -35,5 +35,5 @@
 	<xacro:ros_control_guardian namespace="/guardian_terabot"/>
 	<xacro:terabot name="terabot" parent="base_link">
-		<origin xyz="0.100 0 0.375" rpy="0 0 0"/>
+		<origin xyz="0.190 0 0.287" rpy="0 0 0"/>
 	</xacro:terabot>
 </robot>
